Commit message: removing table object from scene

File: urdf/ur.urdf.xacro (robot description, xacro)
@@ -55,5 +55,5 @@
    <xacro:if value="${is_sim_gazebo or is_sim_ignition}">
      <link name="ground_plane">
-       <visual>
+       <!-- <visual>
          <origin rpy="0 0 0" xyz="0 0 0"/>
          <geometry>
@@ -69,5 +69,5 @@
            <box size="5 5 0"/>
          </geometry>
-       </collision>
+       </collision> -->
      </link>
      <joint name="ground_plane_joint" type="fixed">
