Commit message: adjusting the code to suit gemma setup

File: urdf/ur_macro.xacro (robot description, xacro)
@@ -318,5 +318,5 @@
       <xacro:insert_block name="origin" />
       <parent link="${parent}" />
-      <child link="${tf_prefix}base_link" />
+      <child link="${tf_prefix}table" />
     </joint>
     <!-- joints - main serial chain -->
@@ -436,11 +436,88 @@
       <origin xyz="0 0 0" rpy="0 ${-pi/2.0} ${-pi/2.0}" />
     </joint>
-    <!-- ROS-Industrial 'tool0' frame - all-zeros tool frame -->
-    <link name="${tf_prefix}tool0"/>
-    <joint name="${tf_prefix}flange-tool0" type="fixed">
-      <!-- default toolframe - X+ left, Y+ up, Z+ front -->
-      <origin xyz="0 0 0" rpy="${pi/2.0} 0 ${pi/2.0}"/>
+    <link name="${tf_prefix}tool_temp">
+      <visual>
+        <origin xyz="0 0 0" rpy="0 0 0" />
+        <geometry>
+          <xacro:get_mesh name="ee" type="visual"/>
+        </geometry>
+        <material name="temptu_airpod_gripper">
+          <color rgba="${100.0/255.0} ${100.0/255.0} ${100.0/255.0} 1" />
+        </material>
+      </visual>
+      <collision>
+        <origin xyz="0 0 0" rpy="0 0 0" />
+        <geometry>
+          <xacro:get_mesh name="ee" type="collision"/>
+        </geometry>
+      </collision>
+    </link>
+    <joint name="${tf_prefix}flange-tool_temp" type="fixed">
+      <origin xyz="0 0 0" rpy="-${pi/2.0} 0 -${pi/2.0}"/>
       <parent link="${tf_prefix}flange"/>
+      <child link="${tf_prefix}tool_temp"/>
+    </joint>
+    <link name="${tf_prefix}camera_ee" />
+    <joint name="${tf_prefix}tool_temp-camera_ee" type="fixed">
+      <origin xyz="0.006835956674082612 -0.04985659335752479 0.0976500318266122" rpy="0 0 0"/>
+      <parent link="${tf_prefix}tool_temp"/>
+      <child link="${tf_prefix}camera_ee"/>
+    </joint>
+	<xacro:property name="airbrush_calib_x_angle" value="-0.009598"/>
+	<xacro:property name="airbrush_calib_y_angle" value="-0.008347"/>
+	<xacro:property name="airbrush_calib_x_shift" value="0.001816"/>
+	<xacro:property name="airbrush_calib_y_shift" value="-0.005313"/>
+	<xacro:property name="airbrush_calib_z_shift" value="-0.006385"/>
+    <link name="${tf_prefix}tool0_no_calib" />
+    <joint name="${tf_prefix}tool_temp-tool0_no_calib" type="fixed">
+      <origin xyz="0 0 0.1352" rpy="0 0 0"/>
+      <parent link="${tf_prefix}tool_temp"/>
+      <child link="${tf_prefix}tool0_no_calib"/>
+    </joint>
+    <link name="${tf_prefix}tool0" />
+    <joint name="${tf_prefix}tool0_no_calib-tool0" type="fixed">
+      <origin xyz="${-1.0 * airbrush_calib_x_shift} ${airbrush_calib_y_shift} ${airbrush_calib_z_shift}" rpy="${-1.0 * airbrush_calib_y_angle} ${-1.0 * airbrush_calib_x_angle} 0"/>
+      <parent link="${tf_prefix}tool0_no_calib"/>
       <child link="${tf_prefix}tool0"/>
+    </joint>
+    <link name="${tf_prefix}laser_ee_no_calib" />
+    <joint name="${tf_prefix}tool_temp-laser_ee_no_calib" type="fixed">
+      <origin xyz="0 -0.0665 0.112" rpy="0 0 0"/>
+      <parent link="${tf_prefix}tool_temp"/>
+      <child link="${tf_prefix}laser_ee_no_calib"/>
+    </joint>
+    <xacro:property name="laser_calib_x_angle" value="0.0"/>
+    <xacro:property name="laser_calib_y_angle" value="0.0"/>
+    <xacro:property name="laser_calib_x_shift" value="0.0"/>
+    <xacro:property name="laser_calib_y_shift" value="0.0"/>
+    <xacro:property name="laser_calib_z_shift" value="0.0"/>
+    <link name="${tf_prefix}laser_ee" />
+    <joint name="${tf_prefix}laser_ee_no_calib-laser_ee" type="fixed">
+      <origin xyz="${-1.0 * laser_calib_x_shift} ${laser_calib_y_shift} ${laser_calib_z_shift}" rpy="${-1.0 * laser_calib_y_angle} ${-1.0 * laser_calib_x_angle} 0"/>
+      <parent link="${tf_prefix}laser_ee_no_calib"/>
+      <child link="${tf_prefix}laser_ee"/>
+    </joint>
+    <xacro:property name="table_height" value="0.77"/>
+    <xacro:property name="face_x" value="0"/>
+    <xacro:property name="face_y" value="-0.70"/>
+    <xacro:property name="face_z" value="0.45"/>
+    <link name="${tf_prefix}table">
+      <visual>
+        <origin xyz="0 0 ${table_height}" rpy="0 0 0" />
+        <geometry>
+          <xacro:get_mesh name="table" type="visual"/>
+        </geometry>
+      </visual>
+      <collision>
+        <origin xyz="0 0 ${table_height}" rpy="0 0 0" />
+        <geometry>
+          <xacro:get_mesh name="table" type="collision"/>
+        </geometry>
+      </collision>
+    </link>
+    <joint name="${tf_prefix}table-base_link" type="fixed">
+      <origin xyz="0 0 ${table_height}" rpy="0 0 0"/>
+      <parent link="${tf_prefix}table"/>
+      <child link="${tf_prefix}base_link"/>
     </joint>
   </xacro:macro>

Commit message: .

File: urdf/ur_macro.xacro (robot description, xacro)
@@ -464,4 +464,35 @@
       <child link="${tf_prefix}camera_ee"/>
     </joint>
+  <link name="${tf_prefix}cms_marker">
+    <visual>
+      <origin xyz="0 0 0" rpy="0 0 0" />
+      <geometry>
+        <xacro:get_mesh name="cms" type="visual"/>
+      </geometry>
+    </visual>
+    <collision>
+      <origin xyz="0 0 0" rpy="0 0 0" />
+      <geometry>
+        <xacro:get_mesh name="cms" type="collision"/>
+      </geometry>
+    </collision>
+  </link>
+  <joint name="${tf_prefix}base_link-cms_marker" type="fixed">
+    <!-- cms label --> <origin xyz="-0.5 0.3 0.4" rpy="${90*(pi/180)} 0 ${45*(pi/180)}"/>
+    <parent link="${tf_prefix}base_link"/>
+    <child link="${tf_prefix}cms_marker"/>
+  </joint>
+  <link name="${tf_prefix}cms_backbubbling" />
+  <joint name="${tf_prefix}cms_marker-cms_backbubbling" type="fixed">
+    <origin xyz="0.053 -0.11736 -0.05377" rpy="${56*(pi/180)} 0 0"/>
+    <parent link="${tf_prefix}cms_marker"/>
+    <child link="${tf_prefix}cms_backbubbling"/>
+  </joint>
+  <link name="${tf_prefix}cms_purging" />
+  <joint name="${tf_prefix}cms_marker-cms_purging" type="fixed">
+    <origin xyz="-0.032 -0.11736 -0.05377" rpy="${56*(pi/180)} 0 0"/>
+    <parent link="${tf_prefix}cms_marker"/>
+    <child link="${tf_prefix}cms_purging"/>
+  </joint>
 	<xacro:property name="airbrush_calib_x_angle" value="-0.009598"/>
 	<xacro:property name="airbrush_calib_y_angle" value="-0.008347"/>

Commit message: .

File: urdf/ur_macro.xacro (robot description, xacro)
@@ -485,5 +485,5 @@
   <link name="${tf_prefix}cms_backbubbling" />
   <joint name="${tf_prefix}cms_marker-cms_backbubbling" type="fixed">
-    <origin xyz="0.053 -0.11736 -0.05377" rpy="${56*(pi/180)} 0 0"/>
+    <origin xyz="0.053 -0.11736 -0.05377" rpy="${(-34)*(pi/180)} 0 0"/>
     <parent link="${tf_prefix}cms_marker"/>
     <child link="${tf_prefix}cms_backbubbling"/>
@@ -491,7 +491,13 @@
   <link name="${tf_prefix}cms_purging" />
   <joint name="${tf_prefix}cms_marker-cms_purging" type="fixed">
-    <origin xyz="-0.032 -0.11736 -0.05377" rpy="${56*(pi/180)} 0 0"/>
+    <origin xyz="-0.032 -0.11736 -0.05377" rpy="${(-34)*(pi/180)} 0 0"/>
     <parent link="${tf_prefix}cms_marker"/>
     <child link="${tf_prefix}cms_purging"/>
+  </joint>
+  <link name="${tf_prefix}cms_brush" />
+  <joint name="${tf_prefix}cms_marker-cms_brush" type="fixed">
+    <origin xyz="0.07 -0.06 0.05" rpy="0 0 0"/>
+    <parent link="${tf_prefix}cms_marker"/>
+    <child link="${tf_prefix}cms_brush"/>
   </joint>
 	<xacro:property name="airbrush_calib_x_angle" value="-0.009598"/>
@@ -512,4 +518,10 @@
       <child link="${tf_prefix}tool0"/>
     </joint>
+    <link name="${tf_prefix}paint_cup_ee" />
+    <joint name="${tf_prefix}tool_temp-paint_cup_ee" type="fixed">
+      <origin xyz="0 0 0.07" rpy="0 0 0"/>
+      <parent link="${tf_prefix}tool_temp"/>
+      <child link="${tf_prefix}paint_cup_ee"/>
+    </joint>
     <link name="${tf_prefix}laser_ee_no_calib" />
     <joint name="${tf_prefix}tool_temp-laser_ee_no_calib" type="fixed">

Commit message: .

File: urdf/ur_macro.xacro (robot description, xacro)
@@ -485,5 +485,5 @@
   <link name="${tf_prefix}cms_backbubbling" />
   <joint name="${tf_prefix}cms_marker-cms_backbubbling" type="fixed">
-    <origin xyz="0.053 -0.11736 -0.05377" rpy="${(-34)*(pi/180)} 0 0"/>
+    <origin xyz="0 -0.16019 -0.03016" rpy="${(-34)*(pi/180)} 0 0"/>
     <parent link="${tf_prefix}cms_marker"/>
     <child link="${tf_prefix}cms_backbubbling"/>
@@ -497,5 +497,5 @@
   <link name="${tf_prefix}cms_brush" />
   <joint name="${tf_prefix}cms_marker-cms_brush" type="fixed">
-    <origin xyz="0.07 -0.06 0.05" rpy="0 0 0"/>
+    <origin xyz="0.10196 -0.0565 0.01054" rpy="0 0 0"/>
     <parent link="${tf_prefix}cms_marker"/>
     <child link="${tf_prefix}cms_brush"/>
@@ -520,5 +520,5 @@
     <link name="${tf_prefix}paint_cup_ee" />
     <joint name="${tf_prefix}tool_temp-paint_cup_ee" type="fixed">
-      <origin xyz="0 0 0.07" rpy="0 0 0"/>
+      <origin xyz="0 0.016 0.09088" rpy="0 0 0"/>
       <parent link="${tf_prefix}tool_temp"/>
       <child link="${tf_prefix}paint_cup_ee"/>

Commit message: .

File: urdf/ur_macro.xacro (robot description, xacro)
@@ -497,16 +497,16 @@
   <link name="${tf_prefix}cms_brush" />
   <joint name="${tf_prefix}cms_marker-cms_brush" type="fixed">
-    <origin xyz="0.10196 -0.0565 0.01054" rpy="0 0 0"/>
+    <origin xyz="0.10196 -0.0565 -0.01054" rpy="0 0 0"/>
     <parent link="${tf_prefix}cms_marker"/>
     <child link="${tf_prefix}cms_brush"/>
   </joint>
-	<xacro:property name="airbrush_calib_x_angle" value="-0.009598"/>
-	<xacro:property name="airbrush_calib_y_angle" value="-0.008347"/>
-	<xacro:property name="airbrush_calib_x_shift" value="0.001816"/>
-	<xacro:property name="airbrush_calib_y_shift" value="-0.005313"/>
-	<xacro:property name="airbrush_calib_z_shift" value="-0.006385"/>
+	<xacro:property name="airbrush_calib_x_angle" value="0.0"/>
+	<xacro:property name="airbrush_calib_y_angle" value="0.0"/>
+	<xacro:property name="airbrush_calib_x_shift" value="0.0"/>
+	<xacro:property name="airbrush_calib_y_shift" value="0.0"/>
+	<xacro:property name="airbrush_calib_z_shift" value="0.0"/>
     <link name="${tf_prefix}tool0_no_calib" />
     <joint name="${tf_prefix}tool_temp-tool0_no_calib" type="fixed">
-      <origin xyz="0 0 0.1352" rpy="0 0 0"/>
+      <origin xyz="0 0 0.130" rpy="0 0 0"/>
       <parent link="${tf_prefix}tool_temp"/>
       <child link="${tf_prefix}tool0_no_calib"/>
@@ -520,5 +520,5 @@
     <link name="${tf_prefix}paint_cup_ee" />
     <joint name="${tf_prefix}tool_temp-paint_cup_ee" type="fixed">
-      <origin xyz="0 0.016 0.09088" rpy="0 0 0"/>
+      <origin xyz="0 0.016 0.10088" rpy="0 0 0"/>
       <parent link="${tf_prefix}tool_temp"/>
       <child link="${tf_prefix}paint_cup_ee"/>

Commit message: update EE

File: urdf/ur_macro.xacro (robot description, xacro)
@@ -460,5 +460,5 @@
     <link name="${tf_prefix}camera_ee" />
     <joint name="${tf_prefix}tool_temp-camera_ee" type="fixed">
-      <origin xyz="0.006835956674082612 -0.04985659335752479 0.0976500318266122" rpy="0 0 0"/>
+      <origin xyz="0.009 -0.023 0.107" rpy="0 0 0"/>
       <parent link="${tf_prefix}tool_temp"/>
       <child link="${tf_prefix}camera_ee"/>
@@ -508,5 +508,5 @@
     <link name="${tf_prefix}tool0_no_calib" />
     <joint name="${tf_prefix}tool_temp-tool0_no_calib" type="fixed">
-      <origin xyz="0 0 0.130" rpy="0 0 0"/>
+      <origin xyz="0 0 0.116" rpy="0 0 0"/>
       <parent link="${tf_prefix}tool_temp"/>
       <child link="${tf_prefix}tool0_no_calib"/>
@@ -520,5 +520,5 @@
     <link name="${tf_prefix}paint_cup_ee" />
     <joint name="${tf_prefix}tool_temp-paint_cup_ee" type="fixed">
-      <origin xyz="0 0.016 0.10088" rpy="0 0 0"/>
+      <origin xyz="0 0.022 0.088" rpy="0 0 0"/>
       <parent link="${tf_prefix}tool_temp"/>
       <child link="${tf_prefix}paint_cup_ee"/>
@@ -526,5 +526,5 @@
     <link name="${tf_prefix}laser_ee_no_calib" />
     <joint name="${tf_prefix}tool_temp-laser_ee_no_calib" type="fixed">
-      <origin xyz="0 -0.0665 0.112" rpy="0 0 0"/>
+      <origin xyz="0.01 -0.009 0.112" rpy="0 0 0"/>
       <parent link="${tf_prefix}tool_temp"/>
       <child link="${tf_prefix}laser_ee_no_calib"/>

Commit message: .

File: urdf/ur_macro.xacro (robot description, xacro)
@@ -485,5 +485,5 @@
   <link name="${tf_prefix}cms_backbubbling" />
   <joint name="${tf_prefix}cms_marker-cms_backbubbling" type="fixed">
-    <origin xyz="0 -0.16019 -0.03016" rpy="${(-34)*(pi/180)} 0 0"/>
+    <origin xyz="0 -0.16 -0.029" rpy="${(-34)*(pi/180)} 0 0"/>
     <parent link="${tf_prefix}cms_marker"/>
     <child link="${tf_prefix}cms_backbubbling"/>
@@ -501,4 +501,10 @@
     <child link="${tf_prefix}cms_brush"/>
   </joint>
+  <link name="${tf_prefix}cms_papper_roll" />
+  <joint name="${tf_prefix}cms_marker-cms_papper_roll" type="fixed">
+    <origin xyz="0.16	-0.115	-0.067" rpy="0 0 0"/>
+    <parent link="${tf_prefix}cms_marker"/>
+    <child link="${tf_prefix}cms_papper_roll"/>
+  </joint>
 	<xacro:property name="airbrush_calib_x_angle" value="0.0"/>
 	<xacro:property name="airbrush_calib_y_angle" value="0.0"/>

Commit message: .

File: urdf/ur_macro.xacro (robot description, xacro)
@@ -479,5 +479,5 @@
   </link>
   <joint name="${tf_prefix}base_link-cms_marker" type="fixed">
-    <!-- cms label --> <origin xyz="-0.5 0.3 0.4" rpy="${90*(pi/180)} 0 ${45*(pi/180)}"/>
+    <!-- cms label --> <origin xyz="-0.674 0.358 0.034" rpy="1.559 -0.011 0.845"/>
     <parent link="${tf_prefix}base_link"/>
     <child link="${tf_prefix}cms_marker"/>

Commit message: .

File: urdf/ur_macro.xacro (robot description, xacro)
@@ -489,4 +489,10 @@
     <child link="${tf_prefix}cms_backbubbling"/>
   </joint>
+  <link name="${tf_prefix}cms_paint_load" />
+  <joint name="${tf_prefix}cms_marker-cms_paint_load" type="fixed">
+    <origin xyz="0	-0.043	-0.025" rpy="0 0 0"/>
+    <parent link="${tf_prefix}cms_marker"/>
+    <child link="${tf_prefix}cms_paint_load"/>
+  </joint>
   <link name="${tf_prefix}cms_purging" />
   <joint name="${tf_prefix}cms_marker-cms_purging" type="fixed">

Commit message: .

File: urdf/ur_macro.xacro (robot description, xacro)
@@ -479,5 +479,5 @@
   </link>
   <joint name="${tf_prefix}base_link-cms_marker" type="fixed">
-    <!-- cms label --> <origin xyz="-0.674 0.358 0.034" rpy="1.559 -0.011 0.845"/>
+    <!-- cms label --> <origin xyz="-0.667 0.357 0.037" rpy="1.561 -0.023 0.848"/>
     <parent link="${tf_prefix}base_link"/>
     <child link="${tf_prefix}cms_marker"/>
@@ -491,5 +491,5 @@
   <link name="${tf_prefix}cms_paint_load" />
   <joint name="${tf_prefix}cms_marker-cms_paint_load" type="fixed">
-    <origin xyz="0	-0.043	-0.025" rpy="0 0 0"/>
+    <origin xyz="0	-0.043	-0.03" rpy="0 0 0"/>
     <parent link="${tf_prefix}cms_marker"/>
     <child link="${tf_prefix}cms_paint_load"/>

Commit message: .

File: urdf/ur_macro.xacro (robot description, xacro)
@@ -479,5 +479,5 @@
   </link>
   <joint name="${tf_prefix}base_link-cms_marker" type="fixed">
-    <!-- cms label --> <origin xyz="-0.667 0.357 0.037" rpy="1.561 -0.023 0.848"/>
+    <!-- cms label --> <origin xyz="-0.667 0.357 0.036" rpy="1.564 -0.017 0.851"/>
     <parent link="${tf_prefix}base_link"/>
     <child link="${tf_prefix}cms_marker"/>

Commit message: .

File: urdf/ur_macro.xacro (robot description, xacro)
@@ -507,9 +507,9 @@
     <child link="${tf_prefix}cms_brush"/>
   </joint>
-  <link name="${tf_prefix}cms_papper_roll" />
-  <joint name="${tf_prefix}cms_marker-cms_papper_roll" type="fixed">
+  <link name="${tf_prefix}cms_paper_roll" />
+  <joint name="${tf_prefix}cms_marker-cms_paper_roll" type="fixed">
     <origin xyz="0.16	-0.115	-0.067" rpy="0 0 0"/>
     <parent link="${tf_prefix}cms_marker"/>
-    <child link="${tf_prefix}cms_papper_roll"/>
+    <child link="${tf_prefix}cms_paper_roll"/>
   </joint>
 	<xacro:property name="airbrush_calib_x_angle" value="0.0"/>

Commit message: .

File: urdf/ur_macro.xacro (robot description, xacro)
@@ -464,4 +464,10 @@
       <child link="${tf_prefix}camera_ee"/>
     </joint>
+  <link name="${tf_prefix}base_face_link" />
+  <joint name="${tf_prefix}base_link-base_face_link" type="fixed">
+    <origin xyz="0 0 0" rpy="0 0 ${(180)*(pi/180)}"/>
+    <parent link="${tf_prefix}base_link"/>
+    <child link="${tf_prefix}base_face_link"/>
+  </joint>
   <link name="${tf_prefix}cms_marker">
     <visual>

Commit message: remove redindant code

File: urdf/ur_macro.xacro (robot description, xacro)
@@ -507,10 +507,4 @@
     <child link="${tf_prefix}cms_purging"/>
   </joint>
-  <link name="${tf_prefix}cms_brush" />
-  <joint name="${tf_prefix}cms_marker-cms_brush" type="fixed">
-    <origin xyz="0.10196 -0.0565 -0.01054" rpy="0 0 0"/>
-    <parent link="${tf_prefix}cms_marker"/>
-    <child link="${tf_prefix}cms_brush"/>
-  </joint>
   <link name="${tf_prefix}cms_paper_roll" />
   <joint name="${tf_prefix}cms_marker-cms_paper_roll" type="fixed">
